File: logic.sch (EAGLE design)
At the start: 14 parts, among them CON1 PINHEAD_1X10-2, CON2 PINHEAD_1X10-2, CON3 CON-4P-JST_GH-RA, CON8 CON-4P-JST_GH-RA, IC3 TJA1051

Commit message: silk updates
Parts:
- added U$2: CONNECTION, usb2can_master_lib:CONNECTION
Connections:
- removed net GAIN_OUT: MODULE2.GAIN_OUT
- removed net GATE_ENABLE_OUT: MODULE2.GATE_ENABLE_OUT
- removed net GPIO1: MODULE2.GPIO2
- removed net GPIO2: MODULE2.GPIO1
- net GND: now also U$2.P$1
- net GNDD: now also U$2.P$2
Other:
- moved on the sheet: LED1, LED2, R10, R11, R12, R13
