File: option2/logic.brd (EAGLE design)
At the start: 37 x 36 mm, 16 parts, among them CON1 PINHEAD_1X10-2, CON2 PINHEAD_1X10-2, CON3 CON-4P-JST_GH-RA, CON8 CON-4P-JST_GH-RA, IC3 TJA1051

Commit message: updates here and there
Parts:
- added CON4: PINHEAD_1X03-2.54-RA, pinhead:1X03-PTH-2.54-RA
- moved U$2 3.00 mm to (4.53, -17.5)
- moved C11 3.00 mm to (-2.50, -15.4)
- moved CON3 3.00 mm to (0.00, -21.6)
- moved CON8 3.00 mm to (0.00, -21.6)
- moved IC3 3.00 mm to (0.20, -15.5)
- moved LED1 3.00 mm to (5.50, -21.3)
- moved LED2 3.00 mm to (-5.50, -21.0)
- moved R10 3.00 mm to (5.50, -19.1)
- moved R11 3.00 mm to (4.42, -15.2)
- moved R12 3.00 mm to (3.38, -15.2)
- moved R13 3.00 mm to (-3.55, -15.4)
- moved R7 3.00 mm to (-4.85, -15.4)
Routing:
- net CAN1_RX: track 24.4 -> 18.8 mm, vias 2 -> 1
- net LED_GREEN: track 5.28 -> 0.54 mm
- net LED_RED: track 2.68 -> 5.84 mm
- net N$28: track 5.96 -> 2.85 mm
- net CAN1_TX: track 24.8 -> 21.8 mm
- net N$18: track 4.12 -> 7.12 mm
- net CAN1_LED: track 10.8 -> 13.8 mm
- net N$6: track 4.33 -> 1.66 mm
- net VDD_5V: track 74.6 -> 76.4 mm
- net N$60: track 17.6 -> 19.2 mm
- net N$35: track 6.92 -> 5.42 mm, vias 1 -> 0
- net N$23: track 11.2 -> 10.2 mm
Other:
- board size 37 x 36 mm -> 37.4 x 38.5 mm
