File: option2/logic.sch (EAGLE design)
At the start: 15 parts, among them CON1 PINHEAD_1X10-2, CON2 PINHEAD_1X10-2, CON3 CON-4P-JST_GH-RA, CON8 CON-4P-JST_GH-RA, IC3 TJA1051

Commit message: updates here and there
Parts:
- added CON4: PINHEAD_1X03-2.54-RA, pinhead:PINHEAD_1X03-2.54-RA
Changed lines of the file:
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@@
 <part name="CON1" library="pinhead" library_urn="urn:adsk.eagle:library:2540341" deviceset="PINHEAD_1X10" device="-2" package3d_urn="urn:adsk.eagle:package:6503373/2"/>
 <part name="CON2" library="pinhead" library_urn="urn:adsk.eagle:library:2540341" deviceset="PINHEAD_1X10" device="-2" package3d_urn="urn:adsk.eagle:package:6503373/2"/>
-<part name="MODULE2" library="zubax_modules" library_urn="urn:adsk.eagle:library:5014895" deviceset="MITOHONDRIQUE" device="-TH" package3d_urn="urn:adsk.eagle:package:4410646/9"/>
+<part name="MODULE2" library="zubax_modules" library_urn="urn:adsk.eagle:library:5014895" deviceset="MITOHONDRIQUE" device="-TH" package3d_urn="urn:adsk.eagle:package:4410646/10"/>
 <part name="CON3" library="Connectors" library_urn="urn:adsk.eagle:library:3750510" deviceset="CON-4P" device="-RA" package3d_urn="urn:adsk.eagle:package:1040150/5" technology="-JST_GH"/>
 <part name="IC3" library="myxa_masterlib" library_urn="urn:adsk.eagle:library:1040030" deviceset="TJA1051" device="" package3d_urn="urn:adsk.eagle:package:1040194/3"/>
@@
 <part name="U$2" library="usb2can_master_lib" deviceset="CONNECTION" device=""/>
 <part name="GND2" library="supply_symbols" library_urn="urn:adsk.eagle:library:5017758" deviceset="GND" device="" value="GND"/>
+<part name="CON4" library="pinhead" library_urn="urn:adsk.eagle:library:2540341" deviceset="PINHEAD_1X03" device="-2.54-RA" package3d_urn="urn:adsk.eagle:package:6650270/2"/>
 </parts>
 <sheets>
@@
 <attribute name="VALUE" x="302.26" y="105.41" size="1.27" layer="96" font="vector" ratio="15" align="center"/>
 </instance>
+<instance part="CON4" gate="G$1" x="205.74" y="78.74" smashed="yes">
+<attribute name="NAME" x="208.28" y="90.17" size="1.778" layer="95" font="vector" ratio="15" align="center"/>
+</instance>
 </instances>
