File: option2/powerstage.sch (EAGLE design)
At the start: 38 parts, among them CON1 PINHEAD_1X10-2-FEMALE, CON2 BATTERY_CON-2P-XT30-RA, CON3 PINHEAD_1X10-2-FEMALE, IC5 MCP9700, Q1 BUK7K6R2-40EX, Q2 BUK7K6R2-40EX, Q3 BUK7K6R2-40EX

Commit message: updates here and there
Parts:
- removed D3, D4: PTVS36VP1UP,115-36V-SOD128, TVS_diodes:PTVS36VP1UP,115-36V-SOD128
Connections:
- net PGND: no longer D3.A, D4.A
- net VDC: no longer D3.C, D4.C
Changed lines of the file:
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@@
 <part name="+P2" library="supply_symbols" library_urn="urn:adsk.eagle:library:5017758" deviceset="VDC" device=""/>
 <part name="GND5" library="supply_symbols" library_urn="urn:adsk.eagle:library:5017758" deviceset="PGND" device="" value="PGND"/>
-<part name="D3" library="TVS_diodes" library_urn="urn:adsk.eagle:library:3333632" deviceset="PTVS36VP1UP,115" device="-SOD128" package3d_urn="urn:adsk.eagle:package:6533206/2" technology="-36V"/>
-<part name="D4" library="TVS_diodes" library_urn="urn:adsk.eagle:library:3333632" deviceset="PTVS36VP1UP,115" device="-SOD128" package3d_urn="urn:adsk.eagle:package:6533206/2" technology="-36V"/>
 </parts>
 <sheets>
@@
 <attribute name="VALUE" x="167.64" y="156.21" size="1.27" layer="97" font="vector" ratio="15" align="center"/>
 </instance>
-<instance part="D3" gate="G$1" x="109.22" y="226.06" smashed="yes" rot="R90">
-<attribute name="NAME" x="106.68" y="226.06" size="1.27" layer="95" font="vector" ratio="15" rot="R90" align="center"/>
-<attribute name="MANF#" x="111.76" y="226.06" size="1.016" layer="95" font="vector" ratio="15" rot="R90" align="center"/>
-</instance>
-<instance part="D4" gate="G$1" x="119.38" y="226.06" smashed="yes" rot="R90">
-<attribute name="NAME" x="116.84" y="226.06" size="1.27" layer="95" font="vector" ratio="15" rot="R90" align="center"/>
-<attribute name="MANF#" x="121.92" y="226.06" size="1.016" layer="95" font="vector" ratio="15" rot="R90" align="center"/>
-</instance>
 </instances>
 <busses>
@@
 <wire x1="45.72" y1="226.06" x2="45.72" y2="220.98" width="0.1524" layer="91"/>
 <wire x1="45.72" y1="220.98" x2="48.26" y2="220.98" width="0.1524" layer="91"/>
-<wire x1="104.14" y1="220.98" x2="109.22" y2="220.98" width="0.1524" layer="91"/>
-<junction x="104.14" y="220.98"/>
-<pinref part="D3" gate="G$1" pin="A"/>
-<wire x1="109.22" y1="220.98" x2="109.22" y2="223.52" width="0.1524" layer="91"/>
-<wire x1="109.22" y1="220.98" x2="119.38" y2="220.98" width="0.1524" layer="91"/>
-<junction x="109.22" y="220.98"/>
-<pinref part="D4" gate="G$1" pin="A"/>
-<wire x1="119.38" y1="220.98" x2="119.38" y2="223.52" width="0.1524" layer="91"/>
 </segment>
 <segment>
@@
 <wire x1="45.72" y1="228.6" x2="45.72" y2="233.68" width="0.1524" layer="91"/>
 <wire x1="45.72" y1="233.68" x2="48.26" y2="233.68" width="0.1524" layer="91"/>
-<wire x1="104.14" y1="233.68" x2="109.22" y2="233.68" width="0.1524" layer="91"/>
-<junction x="104.14" y="233.68"/>
-<pinref part="D3" gate="G$1" pin="C"/>
-<wire x1="109.22" y1="231.14" x2="109.22" y2="228.6" width="0.1524" layer="91"/>
-<pinref part="D4" gate="G$1" pin="C"/>
-<wire x1="119.38" y1="231.14" x2="119.38" y2="228.6" width="0.1524" layer="91"/>
-<wire x1="109.22" y1="233.68" x2="109.22" y2="231.14" width="0.1524" layer="91"/>
-<wire x1="109.22" y1="233.68" x2="119.38" y2="233.68" width="0.1524" layer="91"/>
-<junction x="109.22" y="233.68"/>
-<wire x1="119.38" y1="233.68" x2="119.38" y2="231.14" width="0.1524" layer="91"/>
-</segment>
-<segment>
+</segment>
+<segment>
