File: option1/connectors.brd (EAGLE design)
At the start: 13 x 14.5 mm, 14 parts, among them CON1 PINHEAD_1X06-2, CON2 PINHEAD_1X03-2.54-RA, CON3 CON-4P-JST_GH-RA, CON4 PINHEAD_1X02-2, CON5 PINHEAD_1X02-2, CON8 CON-4P-JST_GH-RA, IC3 TJA1051

Commit message: updates here and there
Other:
- outline, holes or cut-outs redrawn
Changed lines of the file:
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@@
 <setting verticaltext="up"/>
 </settings>
-<grid distance="0.05" unitdist="mm" unit="mm" style="lines" multiple="1" display="no" altdistance="5" altunitdist="mil" altunit="mil"/>
+<grid distance="0.5" unitdist="mm" unit="mm" style="lines" multiple="1" display="no" altdistance="5" altunitdist="mil" altunit="mil"/>
 <layers>
 <layer number="1" name="Top" color="4" fill="1" visible="yes" active="yes"/>
@@
 <layer number="14" name="Route14" color="22" fill="1" visible="no" active="no"/>
 <layer number="15" name="Route15" color="23" fill="1" visible="no" active="no"/>
-<layer number="16" name="Bottom" color="1" fill="1" visible="yes" active="yes"/>
-<layer number="17" name="Pads" color="2" fill="1" visible="yes" active="yes"/>
-<layer number="18" name="Vias" color="2" fill="1" visible="yes" active="yes"/>
-<layer number="19" name="Unrouted" color="6" fill="1" visible="yes" active="yes"/>
+<layer number="16" name="Bottom" color="1" fill="1" visible="no" active="yes"/>
+<layer number="17" name="Pads" color="2" fill="1" visible="no" active="yes"/>
+<layer number="18" name="Vias" color="2" fill="1" visible="no" active="yes"/>
+<layer number="19" name="Unrouted" color="6" fill="1" visible="no" active="yes"/>
 <layer number="20" name="Dimension" color="24" fill="1" visible="yes" active="yes"/>
 <layer number="21" name="tPlace" color="7" fill="1" visible="yes" active="yes"/>
-<layer number="22" name="bPlace" color="7" fill="1" visible="yes" active="yes"/>
+<layer number="22" name="bPlace" color="7" fill="1" visible="no" active="yes"/>
 <layer number="23" name="tOrigins" color="15" fill="1" visible="yes" active="yes"/>
-<layer number="24" name="bOrigins" color="15" fill="1" visible="yes" active="yes"/>
+<layer number="24" name="bOrigins" color="15" fill="1" visible="no" active="yes"/>
 <layer number="25" name="tNames" color="7" fill="1" visible="yes" active="yes"/>
-<layer number="26" name="bNames" color="7" fill="1" visible="yes" active="yes"/>
-<layer number="27" name="tValues" color="7" fill="1" visible="yes" active="yes"/>
+<layer number="26" name="bNames" color="7" fill="1" visible="no" active="yes"/>
+<layer number="27" name="tValues" color="7" fill="1" visible="no" active="yes"/>
 <layer number="28" name="bValues" color="7" fill="1" visible="no" active="yes"/>
 <layer number="29" name="tStop" color="7" fill="3" visible="no" active="yes"/>
@@
 <layer number="37" name="tTest" color="7" fill="1" visible="no" active="yes"/>
 <layer number="38" name="bTest" color="7" fill="1" visible="no" active="yes"/>
-<layer number="39" name="tKeepout" color="4" fill="11" visible="yes" active="yes"/>
+<layer number="39" name="tKeepout" color="4" fill="11" visible="no" active="yes"/>
 <layer number="40" name="bKeepout" color="1" fill="11" visible="no" active="yes"/>
-<layer number="41" name="tRestrict" color="4" fill="10" visible="yes" active="yes"/>
+<layer number="41" name="tRestrict" color="4" fill="10" visible="no" active="yes"/>
 <layer number="42" name="bRestrict" color="1" fill="10" visible="no" active="yes"/>
 <layer number="43" name="vRestrict" color="2" fill="10" visible="no" active="yes"/>
 <layer number="44" name="Drills" color="7" fill="1" visible="no" active="yes"/>
-<layer number="45" name="Holes" color="7" fill="1" visible="yes" active="yes"/>
+<layer number="45" name="Holes" color="7" fill="1" visible="no" active="yes"/>
 <layer number="46" name="Milling" color="3" fill="1" visible="no" active="yes"/>
 <layer number="47" name="Measures" color="7" fill="1" visible="no" active="yes"/>
 <layer number="48" name="Document" color="7" fill="1" visible="no" active="yes"/>
-<layer number="49" name="Reference" color="7" fill="1" visible="yes" active="yes"/>
+<layer number="49" name="Reference" color="7" fill="1" visible="no" active="yes"/>
 <layer number="50" name="dxf" color="7" fill="1" visible="no" active="no"/>
 <layer number="51" name="tDocu" color="7" fill="1" visible="yes" active="yes"/>
-<layer number="52" name="bDocu" color="7" fill="1" visible="yes" active="yes"/>
+<layer number="52" name="bDocu" color="7" fill="1" visible="no" active="yes"/>
 <layer number="53" name="tGND_GNDA" color="7" fill="9" visible="no" active="no"/>
 <layer number="54" name="bGND_GNDA" color="1" fill="9" visible="no" active="no"/>
@@
 </layers>
 <board>
-<fusionsync huburn="a.cGVyc29uYWw6dWUyYWE4ZDY4" projecturn="a.cGVyc29uYWw6dWUyYWE4ZDY4IzIwMTgxMTA3MTU4OTYxMDMx" f3durn="urn:adsk.wipprod:dm.lineage:F6T5hmtoRzyO-gJKBP2O0Q" pcbguid="9eefd93a-a020-4737-8592-dac48cb7ff18" lastpulledtime="" lastsyncedchangeguid="2dd12a48-ca80-25c8-6762-f0f654a6b96e"/>
+<fusionsync huburn="a.cGVyc29uYWw6dWUyYWE4ZDY4" projecturn="a.cGVyc29uYWw6dWUyYWE4ZDY4IzIwMTgxMTA4MTU5MTUwNTA2" f3durn="urn:adsk.wipprod:dm.lineage:W-AU7Z-WRBGsUBjO-a_i9g" pcbguid="b2c5e014-5653-4791-840d-ae12ea5a7034" lastpulledtime="2018-11-08T17:53:16Z" lastsyncedchangeguid="92847348-70cf-7b2c-bcb8-8c73375c68d2"/>
 <plain>
 <wire x1="-20" y1="0" x2="0" y2="20" width="0.01" layer="48" curve="-90"/>
@@
 <wire x1="20" y1="-20" x2="-20" y2="-20" width="0.01" layer="48"/>
 <wire x1="-20" y1="-20" x2="-20" y2="0" width="0.01" layer="48"/>
-<wire x1="0.2" y1="-2.5" x2="-5.5" y2="-2.5" width="0.01" layer="20"/>
-<wire x1="-5.5" y1="-2.5" x2="-6.5" y2="-1.5" width="0.01" layer="20" curve="-90"/>
-<wire x1="-6.5" y1="-1.5" x2="-6.5" y2="5.8" width="0.01" layer="20"/>
-<wire x1="-6.5" y1="5.8" x2="-6.5" y2="11" width="0.01" layer="20"/>
-<wire x1="-6.5" y1="11" x2="-5.5" y2="12" width="0.01" layer="20" curve="-90"/>
-<wire x1="-5.5" y1="12" x2="-0.9" y2="12" width="0.01" layer="20"/>
-<wire x1="-0.9" y1="12" x2="5.5" y2="12" width="0.01" layer="20"/>
-<wire x1="5.5" y1="12" x2="6.5" y2="11" width="0.01" layer="20" curve="-90"/>
-<wire x1="6.5" y1="11" x2="6.5" y2="1.6" width="0.01" layer="20"/>
-<wire x1="6.5" y1="1.6" x2="6.5" y2="-1.5" width="0.01" layer="20"/>
-<wire x1="6.5" y1="-1.5" x2="5.5" y2="-2.5" width="0.01" layer="20" curve="-90"/>
-<wire x1="5.5" y1="-2.5" x2="0.2" y2="-2.5" width="0.01" layer="20"/>
+<wire x1="5.5" y1="-2.5" x2="6.5" y2="-1.5" width="0.01" layer="20" curve="90"/>
+<wire x1="6.5" y1="-1.5" x2="6.5" y2="11" width="0.01" layer="20"/>
+<wire x1="6.5" y1="11" x2="5.5" y2="12" width="0.01" layer="20" curve="90"/>
+<wire x1="5.5" y1="12" x2="-5.5" y2="12" width="0.01" layer="20"/>
+<wire x1="-5.5" y1="12" x2="-6.5" y2="11" width="0.01" layer="20" curve="90"/>
+<wire x1="-6.5" y1="11" x2="-6.5" y2="-1.5" width="0.01" layer="20"/>
+<wire x1="-6.5" y1="-1.5" x2="-5.5" y2="-2.5" width="0.01" layer="20" curve="90"/>
+<wire x1="-5.5" y1="-2.5" x2="5.5" y2="-2.5" width="0.01" layer="20"/>
 </plain>
 <attributes>

Commit message: Roting is completed
Parts:
- added R1: 1K, R_digikey:R0402
- moved C11 5.35 mm to (2.95, 5.10), turned to 270 degrees
- moved IC3 0.58 mm to (0.62, 5.10), turned to 180 degrees
Connections:
- removed net LED_GREEN: CON1.4, R12.2
- removed net LED_RED: CON1.3, R13.2
- removed net N$6: CON1.5, R11.2
- new net ADJ: CON1.5, R1.2
- new net BLUE: CON1.6, R11.2
- new net GPIO1: CON1.4, CON2.3
- new net GREEN: CON4.2, R12.2
- new net RED: CON4.1, R13.2
- net CAN1_LED: now also CON1.1; no longer CON1.6
- net CAN1_RX: now also CON1.3; no longer CON5.1
- net CAN1_TX: now also CON1.2; no longer CON5.2
- net GND: now also CON2.1, CON5.1, R1.1; no longer CON4.1
- net VDD_5V: now also CON2.2, CON5.2; no longer CON4.2
Routing:
- net VDD_5V: track 1.97 -> 33.6 mm, vias 1 -> 3
- net CAN1_LED: track 0.00 -> 13.4 mm
- net CAN1_TX: track 0.00 -> 9.61 mm
- net CAN1_RX: track 0.00 -> 8.18 mm
- net N$23: track 1.65 -> 8.69 mm, vias 1 -> 2
- net BLUE: track 0.00 -> 6.72 mm
- net N$35: track 0.31 -> 6.42 mm, vias 0 -> 2
- net ADJ: track 0.00 -> 6.08 mm
- net GPIO1: track 0.00 -> 4.74 mm
- net GREEN: track 0.00 -> 4.48 mm
- net RED: track 0.00 -> 2.04 mm
- net N$28: track 5.90 -> 7.28 mm, vias 2 -> 1
- net GND: track 0.33 -> 1.32 mm, vias 0 -> 10
