File: option1/logic.brd (EAGLE design)
At the start: 37.4 x 33 mm, 8 parts, among them CON1 PINHEAD_1X10-2, CON2 PINHEAD_1X10-2, CON4 PINHEAD_1X02-2, CON5 PINHEAD_1X02-2, CON6 PINHEAD_1X04-2

Commit message: updates here and there
Parts:
- removed R7: 1K, R_digikey:R0402
- added CON3: PINHEAD_1X06-2, pinhead:1X06-PTH-2
- CON6: value PINHEAD_1X04-2 -> PINHEAD_1X02-2; device pinhead:1X04-PTH-2 -> pinhead:1X02-PTH-2
- moved CON6 15.2 mm to (-15.2, -11.6), turned to 135 degrees
Connections:
- removed net N$18: MODULE2.29, R7.1
- new net ADJ: MODULE2.29
- new net GPIO1: MODULE2.27
- new net GPIO2: MODULE2.28
- net GND: no longer R7.2
Routing:
- net CAN1_TX: track 20.2 -> 16.0 mm
- net N$18: track 1.97 -> 0.00 mm
- net CAN1_RX: track 15.7 -> 13.7 mm
Other:
- board size 37.4 x 33 mm -> 37.4 x 32.5 mm

Commit message: Roting is completed
Connections:
- new net BLUE: CON3.1, MODULE2.32
- new net CAN1_LED: CON3.6, MODULE2.36
- new net GREEN: CON4.2, MODULE2.31
- new net RED: CON4.1, MODULE2.30
- net ADJ: now also CON3.2
- net CAN1_RX: now also CON3.4
- net CAN1_TX: now also CON3.5
- net GND: now also CON5.2, CON6.2
- net GPIO1: now also CON3.3, CON6.1
- net VDD_5V: now also CON5.1
Routing:
- net VDD_5V: track 25.2 -> 62.4 mm
- net GPIO1: track 0.00 -> 17.2 mm
- net GREEN: track 0.00 -> 11.1 mm
- net RED: track 0.00 -> 9.83 mm
- net BLUE: track 0.00 -> 9.55 mm
- net CAN1_RX: track 13.7 -> 21.0 mm
- net CAN1_LED: track 0.00 -> 5.12 mm
- net ADJ: track 0.00 -> 3.53 mm
- net CAN1_TX: track 16.0 -> 19.1 mm
